Commit message: Add option to spawn a d435 camera

File: viv_description/urdf/viv_description.urdf.xacro (robot description, xacro)
@@ -1,11 +1,31 @@
 <?xml version="1.0"?>
 <robot xmlns:xacro="http://www.ros.org/wiki/xacro" name="viv">
-    <xacro:property name="M_PI" value="3.1415926535897931" />
+    <!-- Arguments -->
     <xacro:arg name="robot_namespace" default="/" />
+    <xacro:arg name="sim" default="false" />
+    <xacro:property name="sim" value="$(arg sim)" />
+    <xacro:arg name="spawn_d435" default="false" />
+    <xacro:property name="spawn_d435" value="$(arg spawn_d435)" />
     <xacro:include filename="$(find viv_description)/urdf/viv_description_no_ros_control.urdf.xacro" />
-    <gazebo>
-      <plugin name="gazebo_ros_control" filename="libgazebo_ros_control.so">
-        <robotNamespace>$(arg robot_namespace)</robotNamespace>
-      </plugin>
-    </gazebo>
+    <xacro:if value="${sim}">
+      <gazebo>
+        <plugin name="gazebo_ros_control" filename="libgazebo_ros_control.so">
+          <robotNamespace>$(arg robot_namespace)</robotNamespace>
+        </plugin>
+      </gazebo>
+    </xacro:if>
+    <xacro:if value="${spawn_d435}">
+      <xacro:include filename="$(find d435_description)/urdf/d435.xacro" />
+      <joint name="front_camera_joint" type="fixed">
+        <parent link="viv_base"/>
+        <child link="camera_link"/>
+        <origin xyz="${-0.23 + 0.6} 0.2 0.35" rpy="0 0 ${pi/2}" />
+      </joint>
+      <link name="camera_holder_link"/>
+      <joint name="camera_holder_joint" type="fixed">
+        <parent link="viv_base"/>
+        <child link="camera_holder_link"/>
+        <origin xyz="0.0 0.0 0.1" rpy="0 0 0" />
+      </joint>
+    </xacro:if>
 </robot>

Commit message: add rviz, urdf update

File: viv_description/urdf/viv_description.urdf.xacro (robot description, xacro)
@@ -5,5 +5,5 @@
     <xacro:arg name="sim" default="false" />
     <xacro:property name="sim" value="$(arg sim)" />
-    <xacro:arg name="spawn_d435" default="false" />
+    <xacro:arg name="spawn_d435" default="true" />
     <xacro:property name="spawn_d435" value="$(arg spawn_d435)" />
     <xacro:include filename="$(find viv_description)/urdf/viv_description_no_ros_control.urdf.xacro" />
@@ -15,17 +15,3 @@
       </gazebo>
     </xacro:if>
-    <xacro:if value="${spawn_d435}">
-      <xacro:include filename="$(find d435_description)/urdf/d435.xacro" />
-      <joint name="front_camera_joint" type="fixed">
-        <parent link="viv_base"/>
-        <child link="camera_link"/>
-        <origin xyz="${-0.23 + 0.6} 0.2 0.35" rpy="0 0 ${pi/2}" />
-      </joint>
-      <link name="camera_holder_link"/>
-      <joint name="camera_holder_joint" type="fixed">
-        <parent link="viv_base"/>
-        <child link="camera_holder_link"/>
-        <origin xyz="0.0 0.0 0.1" rpy="0 0 0" />
-      </joint>
-    </xacro:if>
 </robot>

File: viv_description/urdf/viv_description_no_ros_control.urdf.xacro (robot description, xacro)
@@ -5,4 +5,6 @@
     <xacro:arg name="sim" default="true" />
     <xacro:property name="sim" value="$(arg sim)" />
+    <xacro:arg name="spawn_d435" default="true" />
+    <xacro:property name="spawn_d435" value="$(arg spawn_d435)" />
     <!--xacro:property name="wheel_radius" value="1" /-->
     <xacro:if value="${sim}">
@@ -333,4 +335,18 @@
       <origin xyz="0 0 0.5" rpy="0 0 0" />
     </joint>
+    <xacro:if value="${spawn_d435}">
+      <xacro:include filename="$(find d435_description)/urdf/d435.xacro" />
+      <joint name="front_camera_joint" type="fixed">
+        <parent link="viv_base"/>
+        <child link="camera_link"/>
+        <origin xyz="${-0.23 + 0.6} 0.2 0.35" rpy="0 0 0" />
+      </joint>
+      <link name="camera_holder_link"/>
+      <joint name="camera_holder_joint" type="fixed">
+        <parent link="viv_base"/>
+        <child link="camera_holder_link"/>
+        <origin xyz="0.0 0.0 0.1" rpy="0 0 0" />
+      </joint>
+    </xacro:if>
     <!-- maka! -->
     <!--gazebo>

Commit message: Use distance to end row for midrow navigation

File: viv_description/urdf/viv_description.urdf.xacro (robot description, xacro)
@@ -5,6 +5,8 @@
     <xacro:arg name="sim" default="false" />
     <xacro:property name="sim" value="$(arg sim)" />
-    <xacro:arg name="spawn_d435" default="true" />
+    <xacro:arg name="spawn_d435" default="false" />
+    <xacro:arg name="spawn_velodyne" default="true" />
     <xacro:property name="spawn_d435" value="$(arg spawn_d435)" />
+    <xacro:property name="spawn_velodyne" value="$(arg spawn_velodyne)" />
     <xacro:include filename="$(find viv_description)/urdf/viv_description_no_ros_control.urdf.xacro" />
     <xacro:if value="${sim}">
@@ -15,3 +17,29 @@
       </gazebo>
     </xacro:if>
+    <xacro:if value="${spawn_d435}">
+      <xacro:include filename="$(find d435_description)/urdf/d435.xacro" />
+      <joint name="front_camera_joint" type="fixed">
+        <parent link="viv_base"/>
+        <child link="camera_link"/>
+        <origin xyz="${-0.23 + 0.6} 0.2 0.35" rpy="0 0 ${pi/2}" />
+      </joint>
+      <link name="camera_holder_link"/>
+      <joint name="camera_holder_joint" type="fixed">
+        <parent link="viv_base"/>
+        <child link="camera_holder_link"/>
+        <origin xyz="0.0 0.0 0.1" rpy="0 0 0" />
+      </joint>
+    </xacro:if>
+    <xacro:if value="${spawn_velodyne}">
+      <xacro:include filename="$(find velodyne_description)/urdf/VLP-16.urdf.xacro" />
+      <xacro:VLP-16 parent="viv_base" name="/rslidar" topic="/rslidar_points" hz="10" samples="440" gpu="false">
+        <origin xyz="0 0 0.4" rpy="0 0 0" />
+      </xacro:VLP-16>
+      <!--link name="velodyne_base_link"/>
+      <joint name="velodyne_joint" type="fixed">
+        <parent link="viv_base"/>
+        <child link="velodyne_base_link"/>
+        <origin xyz="0.0 0.0 0.5" rpy="0 0 ${pi/2}" />
+      </joint-->
+    </xacro:if>
 </robot>
