Commit message: Update models and remove spawn_tank option

File: viv_description/urdf/viv_description_no_ros_control.urdf.xacro (robot description, xacro)
@@ -3,7 +3,7 @@
     <xacro:property name="M_PI" value="3.1415926535897931" />
     <xacro:arg name="robot_namespace" default="/" />
-    <xacro:arg name="spawn_tank" default="true" />
     <link name="viv_base" >
       <visual>
+        <origin xyz="0.0 0 0.1" rpy="0 0 0" />
         <geometry>
           <mesh filename="package://viv_description/meshes/viv_body.dae" />
@@ -76,24 +76,4 @@
       </inertial>
     </link>
-    <xacro:if value="$(eval spawn_tank )">
-      <link name="viv_tank" >
-        <visual>
-          <geometry>
-            <mesh filename="package://viv_description/meshes/viv_tank.dae" />
-          </geometry>
-        </visual>
-        <collision>
-          <origin xyz="0 0 0.15" rpy="0 0 0" />
-          <geometry>
-            <cylinder radius="0.165" length="0.3"/>
-          </geometry>
-        </collision>
-      </link>
-      <joint name="viv_tank_mount_joint" type="fixed">
-        <parent link="viv_base"/>
-        <child link="viv_tank"/>
-        <origin xyz="-0.295 0.0 0.242" rpy="0 0 0" />
-      </joint>
-    </xacro:if>
     <!--wheels-->
     <link name="viv_wheel_front_left" >
@@ -106,5 +86,5 @@
         <origin xyz="0.0 0.0 0.0" rpy="1.57079 0 0" />
         <geometry>
-          <cylinder radius="0.15" length="0.05"/>
+          <cylinder radius="0.14" length="0.05"/>
         </geometry>
       </collision>
@@ -126,5 +106,5 @@
         <origin xyz="0.0 0.0 0.0" rpy="1.57079 0 0" />
         <geometry>
-          <cylinder radius="0.15" length="0.05"/>
+          <cylinder radius="0.14" length="0.05"/>
         </geometry>
       </collision>
@@ -146,5 +126,5 @@
         <origin xyz="0.0 0.0 0.0" rpy="1.57079 0 0" />
         <geometry>
-          <cylinder radius="0.15" length="0.05"/>
+          <cylinder radius="0.14" length="0.05"/>
         </geometry>
       </collision>
@@ -166,5 +146,5 @@
         <origin xyz="0.0 0.0 0.0" rpy="1.57079 0 0" />
         <geometry>
-          <cylinder radius="0.15" length="0.05"/>
+          <cylinder radius="0.14" length="0.05"/>
         </geometry>
       </collision>
@@ -180,5 +160,5 @@
 			<parent link="viv_base"/>
 			<child link="viv_wheel_front_left"/>
-      <origin xyz="0.34 0.294 0.1" rpy="0 0 0" />
+      <origin xyz="0.35 0.3 0.1" rpy="0 0 0" />
 			<axis xyz="0 1 0" rpy="0 0 0"/>
 		</joint>
@@ -186,5 +166,5 @@
 			<parent link="viv_base"/>
 			<child link="viv_wheel_front_right"/>
-      <origin xyz="0.34 -0.294 0.1" rpy="0 0 0" />
+      <origin xyz="0.35 -0.3 0.1" rpy="0 0 0" />
 			<axis xyz="0 1 0" rpy="0 0 0"/>
 		</joint>
@@ -192,5 +172,5 @@
 			<parent link="viv_base"/>
 			<child link="viv_wheel_rear_left"/>
-      <origin xyz="-0.34 0.294 0.1" rpy="0 0 0" />
+      <origin xyz="-0.35 0.3 0.1" rpy="0 0 0" />
 			<axis xyz="0 1 0" rpy="0 0 0"/>
 		</joint>
@@ -198,5 +178,5 @@
 			<parent link="viv_base"/>
 			<child link="viv_wheel_rear_right"/>
-      <origin xyz="-0.34 -0.294 0.1" rpy="0 0 0" />
+      <origin xyz="-0.35 -0.3 0.1" rpy="0 0 0" />
 			<axis xyz="0 1 0" rpy="0 0 0"/>
 		</joint>
@@ -245,5 +225,5 @@
       </visual>
       <collision>
-        <origin xyz="-0.42 0.0 -0.07" rpy="1.57079 0 0" />
+        <origin xyz="-0.42 -0.04 -0.0" rpy="1.57079 0 0" />
         <geometry>
           <cylinder radius="0.05" length="0.05"/>
@@ -258,5 +238,5 @@
       </visual>
       <collision>
-        <origin xyz="-0.42 0.0 -0.07" rpy="1.57079 0 0" />
+        <origin xyz="-0.42 -0.04 -0.0" rpy="1.57079 0 0" />
         <geometry>
           <cylinder radius="0.05" length="0.05"/>
@@ -271,5 +251,5 @@
       </visual>
       <collision>
-        <origin xyz="-0.42 0.0 -0.07" rpy="1.57079 0 0" />
+        <origin xyz="-0.42 -0.04 -0.0" rpy="1.57079 0 0" />
         <geometry>
           <cylinder radius="0.05" length="0.05"/>
@@ -284,5 +264,5 @@
       </visual>
       <collision>
-        <origin xyz="-0.42 0.0 -0.07" rpy="1.57079 0 0" />
+        <origin xyz="-0.42 -0.04 -0.0" rpy="1.57079 0 0" />
         <geometry>
           <cylinder radius="0.05" length="0.05"/>
@@ -293,20 +273,20 @@
       <parent link="viv_base"/>
       <child link="viv_track_1"/>
-      <origin xyz="0.34 0.294 0.1" rpy="0 0 3.14159" />
+      <origin xyz="0.34 0.27 0.1" rpy="0 0 3.14159" />
     </joint>
     <joint name="viv_track_2_mount_joint" type="fixed">
       <parent link="viv_base"/>
       <child link="viv_track_2"/>
-      <origin xyz="0.34 -0.294 0.1" rpy="0 0 3.14159" />
+      <origin xyz="0.34 -0.27 0.1" rpy="3.14159 0 3.14159" />
     </joint>
     <joint name="viv_track_3_mount_joint" type="fixed">
       <parent link="viv_base"/>
       <child link="viv_track_3"/>
-      <origin xyz="-0.34 0.294 0.1" rpy="0 0 0" />
+      <origin xyz="-0.34 0.27 0.1" rpy="3.14159 0 0" />
     </joint>
     <joint name="viv_track_4_mount_joint" type="fixed">
       <parent link="viv_base"/>
       <child link="viv_track_4"/>
-      <origin xyz="-0.34 -0.294 0.1" rpy="0 0 0" />
+      <origin xyz="-0.34 -0.27 0.1" rpy="0 0 0" />
     </joint>
     <!--gazebo reference="viv_wheel_front_left">

Commit message: Flip the viv mesh

File: viv_description/urdf/viv_description_no_ros_control.urdf.xacro (robot description, xacro)
@@ -5,5 +5,5 @@
     <link name="viv_base" >
       <visual>
-        <origin xyz="0.0 0 0.1" rpy="0 0 0" />
+        <origin xyz="0.0 0 0.1" rpy="0 0 3.1415926535897931" />
         <geometry>
           <mesh filename="package://viv_description/meshes/viv_body.dae" />

Commit message: Update urdf to have correct radius for ros_control - TODO fix in simulation

File: viv_description/urdf/viv_description_no_ros_control.urdf.xacro (robot description, xacro)
@@ -86,5 +86,5 @@
         <origin xyz="0.0 0.0 0.0" rpy="1.57079 0 0" />
         <geometry>
-          <cylinder radius="0.14" length="0.05"/>
+          <cylinder radius="0.08" length="0.05"/>
         </geometry>
       </collision>
@@ -106,5 +106,5 @@
         <origin xyz="0.0 0.0 0.0" rpy="1.57079 0 0" />
         <geometry>
-          <cylinder radius="0.14" length="0.05"/>
+          <cylinder radius="0.08" length="0.05"/>
         </geometry>
       </collision>
@@ -126,5 +126,5 @@
         <origin xyz="0.0 0.0 0.0" rpy="1.57079 0 0" />
         <geometry>
-          <cylinder radius="0.14" length="0.05"/>
+          <cylinder radius="0.08" length="0.05"/>
         </geometry>
       </collision>
@@ -146,5 +146,5 @@
         <origin xyz="0.0 0.0 0.0" rpy="1.57079 0 0" />
         <geometry>
-          <cylinder radius="0.14" length="0.05"/>
+          <cylinder radius="0.08" length="0.05"/>
         </geometry>
       </collision>
@@ -160,5 +160,5 @@
 			<parent link="viv_base"/>
 			<child link="viv_wheel_front_left"/>
-      <origin xyz="0.35 0.3 0.1" rpy="0 0 0" />
+      <origin xyz="0.35 0.325 0.1" rpy="0 0 0" />
 			<axis xyz="0 1 0" rpy="0 0 0"/>
 		</joint>
@@ -166,5 +166,5 @@
 			<parent link="viv_base"/>
 			<child link="viv_wheel_front_right"/>
-      <origin xyz="0.35 -0.3 0.1" rpy="0 0 0" />
+      <origin xyz="0.35 -0.325 0.1" rpy="0 0 0" />
 			<axis xyz="0 1 0" rpy="0 0 0"/>
 		</joint>
@@ -172,5 +172,5 @@
 			<parent link="viv_base"/>
 			<child link="viv_wheel_rear_left"/>
-      <origin xyz="-0.35 0.3 0.1" rpy="0 0 0" />
+      <origin xyz="-0.35 0.325 0.1" rpy="0 0 0" />
 			<axis xyz="0 1 0" rpy="0 0 0"/>
 		</joint>
@@ -178,5 +178,5 @@
 			<parent link="viv_base"/>
 			<child link="viv_wheel_rear_right"/>
-      <origin xyz="-0.35 -0.3 0.1" rpy="0 0 0" />
+      <origin xyz="-0.35 -0.325 0.1" rpy="0 0 0" />
 			<axis xyz="0 1 0" rpy="0 0 0"/>
 		</joint>

Commit message: Use sim urdf argument to affect wheel_radius

File: viv_description/urdf/viv_description_no_ros_control.urdf.xacro (robot description, xacro)
@@ -3,4 +3,13 @@
     <xacro:property name="M_PI" value="3.1415926535897931" />
     <xacro:arg name="robot_namespace" default="/" />
+    <xacro:arg name="sim" default="true" />
+    <xacro:property name="sim" value="$(arg sim)" />
+    <!--xacro:property name="wheel_radius" value="1" /-->
+    <xacro:if value="${sim}">
+      <xacro:property name="wheel_radius" value="0.14" />
+    </xacro:if>
+    <xacro:unless value="${sim}">
+      <xacro:property name="wheel_radius" value="0.08" />
+    </xacro:unless>
     <link name="viv_base" >
       <visual>
@@ -86,5 +95,5 @@
         <origin xyz="0.0 0.0 0.0" rpy="1.57079 0 0" />
         <geometry>
-          <cylinder radius="0.08" length="0.05"/>
+          <cylinder radius="${wheel_radius}" length="0.05"/>
         </geometry>
       </collision>
@@ -106,5 +115,5 @@
         <origin xyz="0.0 0.0 0.0" rpy="1.57079 0 0" />
         <geometry>
-          <cylinder radius="0.08" length="0.05"/>
+          <cylinder radius="${wheel_radius}" length="0.05"/>
         </geometry>
       </collision>
@@ -126,5 +135,5 @@
         <origin xyz="0.0 0.0 0.0" rpy="1.57079 0 0" />
         <geometry>
-          <cylinder radius="0.08" length="0.05"/>
+          <cylinder radius="${wheel_radius}" length="0.05"/>
         </geometry>
       </collision>
@@ -146,5 +155,5 @@
         <origin xyz="0.0 0.0 0.0" rpy="1.57079 0 0" />
         <geometry>
-          <cylinder radius="0.08" length="0.05"/>
+          <cylinder radius="${wheel_radius}" length="0.05"/>
         </geometry>
       </collision>

Commit message: Add rslidar link to urdf

File: viv_description/urdf/viv_description_no_ros_control.urdf.xacro (robot description, xacro)
@@ -327,4 +327,10 @@
 			<fdir1 value="1 0 0"/>
 		</gazebo-->
+    <link name="rslidar"/>
+    <joint name="viv_rslidar_mount" type="fixed">
+      <parent link="viv_base"/>
+      <child link="rslidar"/>
+      <origin xyz="0 0 0.5" rpy="0 0 0" />
+    </joint>
     <!-- maka! -->
     <!--gazebo>

Commit message: Add camera mount to urdf

File: viv_description/urdf/viv_description_no_ros_control.urdf.xacro (robot description, xacro)
@@ -333,4 +333,10 @@
       <origin xyz="0 0 0.5" rpy="0 0 0" />
     </joint>
+    <link name="d435_camera_link"/>
+    <joint name="d435_mount" type="fixed">
+      <parent link="viv_base"/>
+      <child link="d435_camera_link"/>
+      <origin xyz="${-0.23 + 0.6} -0.2 0.35" rpy="0 0 0" />
+    </joint>
     <!-- maka! -->
     <!--gazebo>

Commit message: Add base link for mavros

File: viv_description/urdf/viv_description_no_ros_control.urdf.xacro (robot description, xacro)
@@ -341,4 +341,10 @@
       <origin xyz="${-0.23 + 0.6} -0.2 0.35" rpy="0 0 0" />
     </joint>
+    <link name="base_link"/>
+    <joint name="mavros_base_link_mount" type="fixed">
+      <parent link="base_link"/>
+      <child link="viv_base"/>
+      <origin xyz="0 0 -0.55" rpy="0 0 0" />
+    </joint>
     <!-- maka! -->
     <!--gazebo>

Commit message: Add simulation specific navigation code

File: viv_description/urdf/viv_description_no_ros_control.urdf.xacro (robot description, xacro)
@@ -102,5 +102,5 @@
       <inertial>
         <origin xyz="0 0 0"/>
-        <mass value="1"/>
+        <mass value="10"/>
         <inertia ixx="1.0" ixy="0.0" ixz="0.0"
                 iyy="1.0" iyz="0.0"
@@ -122,5 +122,5 @@
       <inertial>
         <origin xyz="0 0 0"/>
-        <mass value="1"/>
+        <mass value="10"/>
         <inertia ixx="1.0" ixy="0.0" ixz="0.0"
                 iyy="1.0" iyz="0.0"
@@ -142,5 +142,5 @@
       <inertial>
         <origin xyz="0 0 0"/>
-        <mass value="1"/>
+        <mass value="10"/>
         <inertia ixx="1.0" ixy="0.0" ixz="0.0"
                 iyy="1.0" iyz="0.0"
@@ -162,5 +162,5 @@
       <inertial>
         <origin xyz="0 0 0"/>
-        <mass value="1"/>
+        <mass value="10"/>
         <inertia ixx="1.0" ixy="0.0" ixz="0.0"
                 iyy="1.0" iyz="0.0"
@@ -301,32 +301,32 @@
       <origin xyz="-0.34 -0.27 0.1" rpy="0 0 0" />
     </joint>
-    <!--gazebo reference="viv_wheel_front_left">
-			<mu1 value="10.0"/>
-			<mu2 value="10.0"/>
-			<kp value="100000.0" />
+    <gazebo reference="viv_wheel_front_left">
+			<mu1 value="2.0"/>
+			<mu2 value="1.0"/>
+			<kp value="10000000.0" />
 			<kd value="1.0" />
 			<fdir1 value="1 0 0"/>
 		</gazebo>
     <gazebo reference="viv_wheel_front_right">
-			<mu1 value="10.0"/>
-			<mu2 value="10.0"/>
-			<kp value="100000.0" />
+			<mu1 value="2.0"/>
+			<mu2 value="1.0"/>
+			<kp value="10000000.0" />
 			<kd value="1.0" />
 			<fdir1 value="1 0 0"/>
 		</gazebo>
     <gazebo reference="viv_wheel_rear_left">
-			<mu1 value="10.0"/>
-			<mu2 value="10.0"/>
-			<kp value="100000.0" />
+			<mu1 value="2.0"/>
+			<mu2 value="1.0"/>
+			<kp value="10000000.0" />
 			<kd value="1.0" />
 			<fdir1 value="1 0 0"/>
 		</gazebo>
     <gazebo reference="viv_wheel_rear_right">
-			<mu1 value="10.0"/>
-			<mu2 value="10.0"/>
-			<kp value="100000.0" />
+			<mu1 value="2.0"/>
+			<mu2 value="1.0"/>
+			<kp value="10000000.0" />
 			<kd value="1.0" />
 			<fdir1 value="1 0 0"/>
-		</gazebo-->
+		</gazebo>
     <link name="rslidar"/>
     <joint name="viv_rslidar_mount" type="fixed">

Commit message: add front and side d435 cam

File: viv_description/urdf/viv_description_no_ros_control.urdf.xacro (robot description, xacro)
@@ -335,9 +335,9 @@
       <origin xyz="0 0 0.5" rpy="0 0 0" />
     </joint>
-    <link name="d435_camera_link"/>
+    <link name="d435_front_link"/>
     <joint name="d435_mount" type="fixed">
       <parent link="viv_base"/>
-      <child link="d435_camera_link"/>
-      <origin xyz="${-0.23 + 0.6} -0.2 0.35" rpy="0 0 0" />
+      <child link="d435_front_link"/>
+      <origin xyz="0.407121 ${0.209 - 0.015} 0.3327" rpy="0 0 0" />
     </joint>
     <link name="base_link"/>

Commit message: Add a more detailed viv model

File: viv_description/urdf/viv_description_no_ros_control.urdf.xacro (robot description, xacro)
@@ -16,7 +16,7 @@
     <link name="viv_base" >
       <visual>
-        <origin xyz="0.0 0 0.1" rpy="0 0 3.1415926535897931" />
-        <geometry>
-          <mesh filename="package://viv_description/meshes/viv_body.dae" />
+        <origin xyz="0.0 0 -0.05" rpy="0 0 0" />
+        <geometry>
+          <mesh filename="package://viv_description/meshes/viv_new_model.dae" />
         </geometry>
       </visual>
@@ -89,9 +89,9 @@
     <!--wheels-->
     <link name="viv_wheel_front_left" >
-      <visual>
+      <!--visual>
         <geometry>
           <mesh filename="package://viv_description/meshes/viv_wheel.dae" />
         </geometry>
-      </visual>
+      </visual-->
       <collision>
         <origin xyz="0.0 0.0 0.0" rpy="1.57079 0 0" />
@@ -109,9 +109,9 @@
     </link>
     <link name="viv_wheel_front_right" >
-      <visual>
+      <!--visual>
         <geometry>
           <mesh filename="package://viv_description/meshes/viv_wheel.dae" />
         </geometry>
-      </visual>
+      </visual-->
       <collision>
         <origin xyz="0.0 0.0 0.0" rpy="1.57079 0 0" />
@@ -129,9 +129,9 @@
     </link>
      <link name="viv_wheel_rear_left" >
-      <visual>
+      <!--visual>
         <geometry>
           <mesh filename="package://viv_description/meshes/viv_wheel.dae" />
         </geometry>
-      </visual>
+      </visual-->
       <collision>
         <origin xyz="0.0 0.0 0.0" rpy="1.57079 0 0" />
@@ -149,9 +149,9 @@
     </link>
     <link name="viv_wheel_rear_right" >
-      <visual>
+      <!--visual>
         <geometry>
           <mesh filename="package://viv_description/meshes/viv_wheel.dae" />
         </geometry>
-      </visual>
+      </visual-->
       <collision>
         <origin xyz="0.0 0.0 0.0" rpy="1.57079 0 0" />
@@ -230,9 +230,9 @@
     <!--tracks-->
     <link name="viv_track_1" >
-      <visual>
+      <!--visual>
         <geometry>
           <mesh filename="package://viv_description/meshes/viv_track.dae" />
         </geometry>
-      </visual>
+      </visual-->
       <collision>
         <origin xyz="-0.42 -0.04 -0.0" rpy="1.57079 0 0" />
@@ -243,9 +243,9 @@
     </link>
     <link name="viv_track_2" >
-      <visual>
+      <!--visual>
         <geometry>
           <mesh filename="package://viv_description/meshes/viv_track.dae" />
         </geometry>
-      </visual>
+      </visual-->
       <collision>
         <origin xyz="-0.42 -0.04 -0.0" rpy="1.57079 0 0" />
@@ -256,9 +256,9 @@
     </link>
      <link name="viv_track_3" >
-      <visual>
+      <!--visual>
         <geometry>
           <mesh filename="package://viv_description/meshes/viv_track.dae" />
         </geometry>
-      </visual>
+      </visual-->
       <collision>
         <origin xyz="-0.42 -0.04 -0.0" rpy="1.57079 0 0" />
@@ -269,9 +269,9 @@
     </link>
     <link name="viv_track_4" >
-      <visual>
+      <!--visual>
         <geometry>
           <mesh filename="package://viv_description/meshes/viv_track.dae" />
         </geometry>
-      </visual>
+      </visual-->
       <collision>
         <origin xyz="-0.42 -0.04 -0.0" rpy="1.57079 0 0" />
